Commit message: Revise sowbot_01.xacro for updated robot design
Updated sowbot_01.xacro to reflect design changes including continuous rubber tracks, chassis modifications, and added components like a mast for GPS and comms.

File: src/agro_robot_sim/urdf/sowbot_01.xacro (robot description, xacro)
@@ -1,52 +1,60 @@
 <?xml version="1.0"?>
-<!--
-  amiga_ng.urdf.xacro  —  Visual URDF for farm-ng Amiga-NG
-  Dimensions sourced from amiga_ros2_description (amiga-ros2-bridge-main).
-  Primitive geometry visual model; no mesh files required.
-  Gazebo Harmonic plugins ported from robo_caatinga.urdf.xacro pattern.
-  Sensor TF positions from amiga_descr.urdf.xacro (relative to base_link):
+<!--sowbot_01.xacro  —  Visual URDF for sowbot
+    • Continuous rubber tracks replace the 4 wheels (visual: long track box + drive/idler rollers)
+    • Chassis split into TWO side body pods sitting above each track
+    • Pods joined by a transverse top frame; vertical mast carries GPS / comms / e-stop
+  Reference dimensions (from supplied RTU.V4 drawing):
+    track ground length   ≈ 1.035 m
+    overall body width     ≈ 0.940 m
+    overall height         ≈ 0.520 m (chassis) + mast
+    track contact width    ≈ 0.242 m (each track)
+  Original Amiga-NG sensor TF positions preserved (relative to base_link):
     GPS (gps_link):   xyz="-0.343  0.273  1.016"
     IMU (bno085):     xyz="-0.300  0.000  0.000"
-    LiDAR:            xyz=" 0.000  0.562  0.141"  (side-mounted, use_lidar:=true)
+    LiDAR:            xyz=" 0.000  0.562  0.141"  (use_lidar:=true)
     OAK-D front:      xyz="-0.248  0.273  0.951"
     OAK-D rear:       xyz="-0.438  0.273  0.951"
-  Wheel geometry from amiga_descr.urdf.xacro:
-    wheel_radius = 0.21717 m
-    wheel z-offset from base_link = -0.4341 m  → base_link rides 0.4341 m above axle centre
-    front axle x = +0.353 / +0.305 m  (slight asymmetry — averaged to 0.329 m)
-    rear  axle x = -0.305 / -0.353 m  (averaged to -0.329 m)
-    track half-width = 0.562 m  → track_width = 1.124 m
-  Plugins (all topics bridged to ROS by ros_gz_bridge):
-    gz-sim-diff-drive-system       cmd_vel → /cmd_vel, odom → /odom
+  Plugins (Gazebo Harmonic; topics bridged by ros_gz_bridge):
+    gz-sim-diff-drive-system       cmd_vel → /cmd_vel, odom → /odom  (skid-steer / track diff)
     gz-sim-joint-state-publisher   joint_states → /joint_states
-    gz-sim-sensors-system          activates gpu_lidar, navsat, imu
-    gz-sim-imu-system
-    gz-sim-navsat-system
+    gz-sim-sensors-system / imu-system / navsat-system
 -->
 <robot xmlns:xacro="http://www.ros.org/wiki/xacro" name="amiga_ng">
-  <!-- ── Amiga-NG dimensions (from amiga_ros2_description) ── -->
-  <xacro:property name="wheel_radius"   value="0.21717"/>
-  <xacro:property name="wheel_width"    value="0.18"/>      <!-- estimated; not in xacro -->
-  <xacro:property name="track_width"    value="1.124"/>     <!-- 2 × 0.562 m -->
-  <xacro:property name="wheelbase"      value="0.658"/>     <!-- 2 × 0.329 m (averaged front/rear asymmetry) -->
-  <xacro:property name="base_link_z"    value="0.4341"/>    <!-- base_link above axle centre -->
-  <!-- Chassis approximation: Amiga body sits above the axle plane -->
-  <xacro:property name="chassis_len"    value="1.10"/>
-  <xacro:property name="chassis_wid"    value="1.20"/>
-  <xacro:property name="chassis_h"      value="0.35"/>
-  <!-- base_link is at axle height; chassis top face is ~base_link_z above axle -->
-  <xacro:property name="chassis_z"      value="${base_link_z - chassis_h/2}"/>
-  <!-- Uprights / frame tubes -->
-  <xacro:property name="upright_h"      value="0.65"/>
-  <xacro:property name="upright_r"      value="0.03"/>
+  <!-- ── Track / chassis dimensions (RTU.V4) ── -->
+  <xacro:property name="track_length"   value="1.035"/>    <!-- ground contact length -->
+  <xacro:property name="track_width"    value="0.242"/>    <!-- each track contact width -->
+  <xacro:property name="track_height"   value="0.22"/>     <!-- track unit vertical extent -->
+  <xacro:property name="drive_radius"   value="0.11"/>     <!-- track roller radius (drive frame) -->
+  <!-- Track centre-to-centre spacing (body width minus one track width) -->
+  <xacro:property name="track_sep"      value="0.698"/>    <!-- 0.940 - 0.242 -->
+  <xacro:property name="track_half"     value="${track_sep/2}"/>
+  <!-- base_link sits at the track roller axle height -->
+  <xacro:property name="base_link_z"    value="${drive_radius}"/>
+  <!-- ── Side body pods (two boxes, one above each track) ── -->
+  <xacro:property name="pod_len"        value="0.95"/>
+  <xacro:property name="pod_wid"        value="0.24"/>
+  <xacro:property name="pod_h"          value="0.30"/>
+  <!-- pod inner face roughly above the track; centre offset = track_half -->
+  <xacro:property name="pod_y"          value="${track_half}"/>
+  <!-- pod vertical centre above base_link (above the track unit) -->
+  <xacro:property name="pod_z"          value="${track_height/2 + pod_h/2}"/>
+  <!-- ── Transverse top frame joining the pods ── -->
+  <xacro:property name="frame_wid"      value="0.94"/>
+  <xacro:property name="frame_len"      value="0.12"/>
+  <xacro:property name="frame_h"        value="0.04"/>
+  <!-- ── Mast (vertical post carrying GPS / comms / e-stop) ── -->
+  <xacro:property name="mast_h"         value="0.55"/>
+  <xacro:property name="mast_r"         value="0.025"/>
   <!-- ── Materials ── -->
   <material name="amiga_green">  <color rgba="0.18 0.42 0.18 1.0"/> </material>
+  <material name="white">        <color rgba="0.88 0.88 0.86 1.0"/> </material>
   <material name="black">        <color rgba="0.10 0.10 0.10 1.0"/> </material>
   <material name="grey">         <color rgba="0.55 0.55 0.55 1.0"/> </material>
   <material name="orange">       <color rgba="1.00 0.50 0.00 1.0"/> </material>
+  <material name="red">          <color rgba="0.80 0.10 0.10 1.0"/> </material>
   <!-- ══════════════════════════════════════════════════════════════
        BASE FRAMES
-       base_footprint  → base_link (raised by wheel_radius so footprint
-       sits on the ground; base_link is at axle-centre height)
+       base_footprint → base_link  (raised by drive_radius so the
+       footprint sits on the ground; base_link at track axle height)
        ══════════════════════════════════════════════════════════════ -->
   <link name="base_footprint"/>
@@ -61,104 +69,28 @@
     <parent link="base_footprint"/>
     <child  link="base_link"/>
-    <origin xyz="0 0 ${wheel_radius}" rpy="0 0 0"/>
-  </joint>
-  <!-- ══════════════════════════════════════════════════════════════
-       CHASSIS BODY
-       Single box approximating the Amiga platform deck.
-       Positioned so its top face aligns with base_link_z above axle.
-       ══════════════════════════════════════════════════════════════ -->
-  <link name="chassis_link">
-    <visual>
-      <origin xyz="0 0 0" rpy="0 0 0"/>
-      <geometry> <box size="${chassis_len} ${chassis_wid} ${chassis_h}"/> </geometry>
-      <material name="amiga_green"/>
-    </visual>
-    <collision>
-      <origin xyz="0 0 0" rpy="0 0 0"/>
-      <geometry> <box size="${chassis_len} ${chassis_wid} ${chassis_h}"/> </geometry>
-    </collision>
-    <inertial>
-      <mass value="120.0"/>
-      <inertia ixx="12.0" ixy="0" ixz="0" iyy="12.0" iyz="0" izz="12.0"/>
-    </inertial>
-  </link>
-  <joint name="chassis_joint" type="fixed">
-    <parent link="base_link"/>
-    <child  link="chassis_link"/>
-    <origin xyz="0 0 ${chassis_z}" rpy="0 0 0"/>
-  </joint>
-  <!-- ══════════════════════════════════════════════════════════════
-       CORNER UPRIGHTS  (4 posts rising from chassis corners)
-       The Amiga has a welded tube frame; approximated with cylinders.
-       ══════════════════════════════════════════════════════════════ -->
-  <xacro:macro name="upright" params="prefix x y">
-    <link name="${prefix}_upright">
+    <origin xyz="0 0 ${base_link_z}" rpy="0 0 0"/>
+  </joint>
+  <!-- ══════════════════════════════════════════════════════════════
+       TRACKS  (left + right)
+       Each track = a long rounded box (rubber belt) plus a drive
+       roller and idler roller for a treaded look. The continuous
+       joint on the drive roller is what the diff-drive plugin spins.
+       ══════════════════════════════════════════════════════════════ -->
+  <xacro:macro name="track" params="prefix y axis_y">
+    <!-- Belt body (visual + collision); fixed to base_link -->
+    <link name="${prefix}_track_link">
       <visual>
         <origin xyz="0 0 0" rpy="0 0 0"/>
-        <geometry> <cylinder radius="${upright_r}" length="${upright_h}"/> </geometry>
-        <material name="grey"/>
+        <geometry> <box size="${track_length} ${track_width} ${track_height}"/> </geometry>
+        <material name="black"/>
       </visual>
       <collision>
         <origin xyz="0 0 0" rpy="0 0 0"/>
-        <geometry> <cylinder radius="${upright_r}" length="${upright_h}"/> </geometry>
-      </collision>
-      <inertial>
-        <mass value="2.0"/>
-        <inertia ixx="0.1" ixy="0" ixz="0" iyy="0.1" iyz="0" izz="0.1"/>
-      </inertial>
-    </link>
-    <joint name="${prefix}_upright_joint" type="fixed">
-      <parent link="chassis_link"/>
-      <child  link="${prefix}_upright"/>
-      <origin xyz="${x} ${y} ${chassis_h/2 + upright_h/2}" rpy="0 0 0"/>
-    </joint>
-  </xacro:macro>
-  <xacro:upright prefix="fl" x=" ${chassis_len/2 - 0.08}" y=" ${chassis_wid/2 - 0.08}"/>
-  <xacro:upright prefix="fr" x=" ${chassis_len/2 - 0.08}" y="-${chassis_wid/2 - 0.08}"/>
-  <xacro:upright prefix="bl" x="-${chassis_len/2 - 0.08}" y=" ${chassis_wid/2 - 0.08}"/>
-  <xacro:upright prefix="br" x="-${chassis_len/2 - 0.08}" y="-${chassis_wid/2 - 0.08}"/>
-  <!-- ══════════════════════════════════════════════════════════════
-       TOP RAIL  (horizontal bar across the top of the uprights)
-       ══════════════════════════════════════════════════════════════ -->
-  <link name="top_rail">
-    <visual>
-      <origin xyz="0 0 0" rpy="0 0 0"/>
-      <geometry> <box size="${chassis_len} ${chassis_wid} 0.04"/> </geometry>
-      <material name="grey"/>
-    </visual>
-    <collision>
-      <origin xyz="0 0 0" rpy="0 0 0"/>
-      <geometry> <box size="${chassis_len} ${chassis_wid} 0.04"/> </geometry>
-    </collision>
-    <inertial>
-      <mass value="5.0"/>
-      <inertia ixx="0.5" ixy="0" ixz="0" iyy="0.5" iyz="0" izz="0.5"/>
-    </inertial>
-  </link>
-  <joint name="top_rail_joint" type="fixed">
-    <parent link="chassis_link"/>
-    <child  link="top_rail"/>
-    <origin xyz="0 0 ${chassis_h/2 + upright_h}" rpy="0 0 0"/>
-  </joint>
-  <!-- ══════════════════════════════════════════════════════════════
-       WHEELS  (4× continuous joints; axis=Y in amiga xacro)
-       Positions from amiga_descr.urdf.xacro joint origins.
-       base_link is at axle height so z=0 for all wheel joints.
-       ══════════════════════════════════════════════════════════════ -->
-  <xacro:macro name="wheel" params="prefix x y axis_y">
-    <link name="${prefix}_wheel_link">
-      <visual>
-        <origin xyz="0 0 0" rpy="${pi/2} 0 0"/>
-        <geometry> <cylinder radius="${wheel_radius}" length="${wheel_width}"/> </geometry>
-        <material name="black"/>
-      </visual>
-      <collision>
-        <origin xyz="0 0 0" rpy="${pi/2} 0 0"/>
-        <geometry> <cylinder radius="${wheel_radius}" length="${wheel_width}"/> </geometry>
+        <geometry> <box size="${track_length} ${track_width} ${track_height}"/> </geometry>
         <surface>
           <friction>
             <ode>
-              <mu>1.5</mu>
-              <mu2>1.5</mu2>
+              <mu>2.0</mu>
+              <mu2>2.0</mu2>
               <fdir1>1 0 0</fdir1>
               <slip1>0.0</slip1>
@@ -169,23 +101,163 @@
       </collision>
       <inertial>
-        <mass value="15.0"/>
-        <inertia ixx="0.7" ixy="0" ixz="0" iyy="0.7" iyz="0" izz="0.7"/>
+        <mass value="18.0"/>
+        <inertia ixx="0.8" ixy="0" ixz="0" iyy="2.0" iyz="0" izz="2.0"/>
       </inertial>
     </link>
-    <joint name="${prefix}_wheel_joint" type="continuous">
+    <joint name="${prefix}_track_joint" type="fixed">
       <parent link="base_link"/>
-      <child  link="${prefix}_wheel_link"/>
-      <origin xyz="${x} ${y} 0" rpy="0 0 0"/>
+      <child  link="${prefix}_track_link"/>
+      <origin xyz="0 ${y} 0" rpy="0 0 0"/>
+    </joint>
+    <!-- Drive roller (front) — the powered, spinning joint -->
+    <link name="${prefix}_drive_link">
+      <visual>
+        <origin xyz="0 0 0" rpy="${pi/2} 0 0"/>
+        <geometry> <cylinder radius="${drive_radius}" length="${track_width}"/> </geometry>
+        <material name="grey"/>
+      </visual>
+      <collision>
+        <origin xyz="0 0 0" rpy="${pi/2} 0 0"/>
+        <geometry> <cylinder radius="${drive_radius}" length="${track_width}"/> </geometry>
+      </collision>
+      <inertial>
+        <mass value="4.0"/>
+        <inertia ixx="0.05" ixy="0" ixz="0" iyy="0.05" iyz="0" izz="0.05"/>
+      </inertial>
+    </link>
+    <joint name="${prefix}_drive_joint" type="continuous">
+      <parent link="base_link"/>
+      <child  link="${prefix}_drive_link"/>
+      <origin xyz="${track_length/2 - drive_radius} ${y} 0" rpy="0 0 0"/>
       <axis xyz="0 ${axis_y} 0"/>
     </joint>
+    <!-- Idler roller (rear) — passive spinning visual -->
+    <link name="${prefix}_idler_link">
+      <visual>
+        <origin xyz="0 0 0" rpy="${pi/2} 0 0"/>
+        <geometry> <cylinder radius="${drive_radius}" length="${track_width}"/> </geometry>
+        <material name="grey"/>
+      </visual>
+      <inertial>
+        <mass value="4.0"/>
+        <inertia ixx="0.05" ixy="0" ixz="0" iyy="0.05" iyz="0" izz="0.05"/>
+      </inertial>
+    </link>
+    <joint name="${prefix}_idler_joint" type="continuous">
+      <parent link="base_link"/>
+      <child  link="${prefix}_idler_link"/>
+      <origin xyz="-${track_length/2 - drive_radius} ${y} 0" rpy="0 0 0"/>
+      <axis xyz="0 ${axis_y} 0"/>
+    </joint>
   </xacro:macro>
-  <!-- Exact x/y from amiga_descr.urdf.xacro; axis_y sign matches original -->
-  <xacro:wheel prefix="front_left"  x=" 0.30508"  y=" 0.56219"  axis_y=" 1"/>
-  <xacro:wheel prefix="front_right" x=" 0.35288"  y="-0.56219"  axis_y="-1"/>
-  <xacro:wheel prefix="rear_left"   x="-0.35312"  y=" 0.56219"  axis_y=" 1"/>
-  <xacro:wheel prefix="rear_right"  x="-0.30507"  y="-0.56219"  axis_y="-1"/>
-  <!-- ══════════════════════════════════════════════════════════════
-       GPS  (from amiga_descr.urdf.xacro: xyz="-0.343 0.273 1.016")
-       Represented as a small box on top of the frame.
+  <xacro:track prefix="left"  y=" ${track_half}" axis_y=" 1"/>
+  <xacro:track prefix="right" y="-${track_half}" axis_y="-1"/>
+  <!-- ══════════════════════════════════════════════════════════════
+       SIDE BODY PODS  (two boxes above the tracks — the split body)
+       ══════════════════════════════════════════════════════════════ -->
+  <xacro:macro name="pod" params="prefix y">
+    <link name="${prefix}_pod_link">
+      <visual>
+        <origin xyz="0 0 0" rpy="0 0 0"/>
+        <geometry> <box size="${pod_len} ${pod_wid} ${pod_h}"/> </geometry>
+        <material name="white"/>
+      </visual>
+      <collision>
+        <origin xyz="0 0 0" rpy="0 0 0"/>
+        <geometry> <box size="${pod_len} ${pod_wid} ${pod_h}"/> </geometry>
+      </collision>
+      <inertial>
+        <mass value="35.0"/>
+        <inertia ixx="3.0" ixy="0" ixz="0" iyy="3.0" iyz="0" izz="3.0"/>
+      </inertial>
+    </link>
+    <joint name="${prefix}_pod_joint" type="fixed">
+      <parent link="base_link"/>
+      <child  link="${prefix}_pod_link"/>
+      <origin xyz="0 ${y} ${pod_z}" rpy="0 0 0"/>
+    </joint>
+  </xacro:macro>
+  <xacro:pod prefix="left"  y=" ${pod_y}"/>
+  <xacro:pod prefix="right" y="-${pod_y}"/>
+  <!-- ══════════════════════════════════════════════════════════════
+       TOP FRAME  (transverse bar joining the two pods)
+       Sits across the top of both pods near the front.
+       ══════════════════════════════════════════════════════════════ -->
+  <link name="top_frame">
+    <visual>
+      <origin xyz="0 0 0" rpy="0 0 0"/>
+      <geometry> <box size="${frame_len} ${frame_wid} ${frame_h}"/> </geometry>
+      <material name="grey"/>
+    </visual>
+    <collision>
+      <origin xyz="0 0 0" rpy="0 0 0"/>
+      <geometry> <box size="${frame_len} ${frame_wid} ${frame_h}"/> </geometry>
+    </collision>
+    <inertial>
+      <mass value="4.0"/>
+      <inertia ixx="0.3" ixy="0" ixz="0" iyy="0.05" iyz="0" izz="0.3"/>
+    </inertial>
+  </link>
+  <joint name="top_frame_joint" type="fixed">
+    <parent link="base_link"/>
+    <child  link="top_frame"/>
+    <origin xyz="${pod_len/2 - 0.15} 0 ${pod_z + pod_h/2 + frame_h/2}" rpy="0 0 0"/>
+  </joint>
+  <!-- ══════════════════════════════════════════════════════════════
+       MAST  (vertical post on the top frame; carries GPS / comms / e-stop)
+       ══════════════════════════════════════════════════════════════ -->
+  <link name="mast_link">
+    <visual>
+      <origin xyz="0 0 0" rpy="0 0 0"/>
+      <geometry> <cylinder radius="${mast_r}" length="${mast_h}"/> </geometry>
+      <material name="grey"/>
+    </visual>
+    <collision>
+      <origin xyz="0 0 0" rpy="0 0 0"/>
+      <geometry> <cylinder radius="${mast_r}" length="${mast_h}"/> </geometry>
+    </collision>
+    <inertial>
+      <mass value="1.5"/>
+      <inertia ixx="0.05" ixy="0" ixz="0" iyy="0.05" iyz="0" izz="0.001"/>
+    </inertial>
+  </link>
+  <!-- Mast mounted on the LEFT pod, near the front corner (one side) -->
+  <joint name="mast_joint" type="fixed">
+    <parent link="left_pod_link"/>
+    <child  link="mast_link"/>
+    <origin xyz="${pod_len/2 - 0.12} 0 ${pod_h/2 + mast_h/2}" rpy="0 0 0"/>
+  </joint>
+  <!-- Comms / control enclosure on the mast (the blue box in the drawing) -->
+  <link name="comms_box">
+    <visual>
+      <origin xyz="0 0 0" rpy="0 0 0"/>
+      <geometry> <box size="0.10 0.14 0.22"/> </geometry>
+      <material name="grey"/>
+    </visual>
+    <inertial>
+      <mass value="1.0"/>
+      <inertia ixx="0.01" ixy="0" ixz="0" iyy="0.01" iyz="0" izz="0.01"/>
+    </inertial>
+  </link>
+  <joint name="comms_box_joint" type="fixed">
+    <parent link="mast_link"/>
+    <child  link="comms_box"/>
+    <origin xyz="0.07 0 0.05" rpy="0 0 0"/>
+  </joint>
+  <!-- E-stop button (the red mushroom on the side) -->
+  <link name="estop_link">
+    <visual>
+      <origin xyz="0 0 0" rpy="0 ${pi/2} 0"/>
+      <geometry> <cylinder radius="0.025" length="0.03"/> </geometry>
+      <material name="red"/>
+    </visual>
+  </link>
+  <joint name="estop_joint" type="fixed">
+    <parent link="left_pod_link"/>
+    <child  link="estop_link"/>
+    <origin xyz="${pod_len/2 - 0.20} ${pod_wid/2} 0.02" rpy="0 0 0"/>
+  </joint>
+  <!-- ══════════════════════════════════════════════════════════════
+       GPS  (xyz="-0.343 0.273 1.016" rel base_link) — preserved
        ══════════════════════════════════════════════════════════════ -->
   <link name="gps_link">
@@ -200,7 +272,7 @@
   </link>
   <joint name="gps_joint" type="fixed">
-    <parent link="base_link"/>
+    <parent link="mast_link"/>
     <child  link="gps_link"/>
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