Commit message: Update sowbot_01.xacro

File: src/agro_robot_sim/urdf/sowbot_01.xacro (robot description, xacro)
@@ -1,5 +1,6 @@
 <?xml version="1.0"?>
-<!--sowbot_01.xacro  —  Visual URDF for sowbot
-    • Continuous rubber tracks replace the 4 wheels (visual: long track box + drive/idler rollers)
+<!--
+  sowbot_urdf.xacro  —
+     • Continuous rubber tracks replace the 4 wheels (visual: long track box + drive/idler rollers)
     • Chassis split into TWO side body pods sitting above each track
     • Pods joined by a transverse top frame; vertical mast carries GPS / comms / e-stop
@@ -34,9 +35,9 @@
   <xacro:property name="pod_len"        value="0.95"/>
   <xacro:property name="pod_wid"        value="0.24"/>
-  <xacro:property name="pod_h"          value="0.30"/>
+  <xacro:property name="pod_h"          value="0.26"/>
   <!-- pod inner face roughly above the track; centre offset = track_half -->
   <xacro:property name="pod_y"          value="${track_half}"/>
-  <!-- pod vertical centre above base_link (above the track unit) -->
-  <xacro:property name="pod_z"          value="${track_height/2 + pod_h/2}"/>
+  <!-- pod vertical centre: drop body so its base overlaps the top of the track unit -->
+  <xacro:property name="pod_z"          value="${track_height/2 + pod_h/2 - 0.05}"/>
   <!-- ── Transverse top frame joining the pods ── -->
   <xacro:property name="frame_wid"      value="0.94"/>
@@ -82,10 +83,10 @@
       <visual>
         <origin xyz="0 0 0" rpy="0 0 0"/>
-        <geometry> <box size="${track_length} ${track_width} ${track_height}"/> </geometry>
+        <geometry> <box size="${track_length - 2*drive_radius} ${track_width} ${track_height}"/> </geometry>
         <material name="black"/>
       </visual>
       <collision>
         <origin xyz="0 0 0" rpy="0 0 0"/>
-        <geometry> <box size="${track_length} ${track_width} ${track_height}"/> </geometry>
+        <geometry> <box size="${track_length - 2*drive_radius} ${track_width} ${track_height}"/> </geometry>
         <surface>
           <friction>
@@ -110,14 +111,14 @@
       <origin xyz="0 ${y} 0" rpy="0 0 0"/>
     </joint>
-    <!-- Drive roller (front) — the powered, spinning joint -->
+    <!-- Drive roller (front) — full track height; forms the rounded front end -->
     <link name="${prefix}_drive_link">
       <visual>
         <origin xyz="0 0 0" rpy="${pi/2} 0 0"/>
-        <geometry> <cylinder radius="${drive_radius}" length="${track_width}"/> </geometry>
-        <material name="grey"/>
+        <geometry> <cylinder radius="${track_height/2}" length="${track_width}"/> </geometry>
+        <material name="black"/>
       </visual>
       <collision>
         <origin xyz="0 0 0" rpy="${pi/2} 0 0"/>
-        <geometry> <cylinder radius="${drive_radius}" length="${track_width}"/> </geometry>
+        <geometry> <cylinder radius="${track_height/2}" length="${track_width}"/> </geometry>
       </collision>
       <inertial>
@@ -132,10 +133,10 @@
       <axis xyz="0 ${axis_y} 0"/>
     </joint>
-    <!-- Idler roller (rear) — passive spinning visual -->
+    <!-- Idler roller (rear) — full track height; forms the rounded rear end -->
     <link name="${prefix}_idler_link">
       <visual>
         <origin xyz="0 0 0" rpy="${pi/2} 0 0"/>
-        <geometry> <cylinder radius="${drive_radius}" length="${track_width}"/> </geometry>
-        <material name="grey"/>
+        <geometry> <cylinder radius="${track_height/2}" length="${track_width}"/> </geometry>
+        <material name="black"/>
       </visual>
       <inertial>
@@ -157,10 +158,38 @@
        ══════════════════════════════════════════════════════════════ -->
   <xacro:macro name="pod" params="prefix y">
+    <!-- Pod profile: a trapezoid in side view — flat bottom (full 0.95), shorter
+         top (0.43), with a FULL-HEIGHT 45° slant face at each end running from the
+         bottom-outer edge up to the top-inner edge, so the slant reaches the very
+         end of the body. Central box (top length, full height) + two thin slant
+         plates covering the slope faces.
+         Literals (no math fns / in-macro properties) for parser compatibility:
+           pod_h=0.26, central box len=0.43, slant_len=0.3677, pitch=0.7854 rad,
+           slant centre x=±0.345 (spans bottom-outer 0.475/-0.13 to top-inner 0.215/+0.13) -->
     <link name="${prefix}_pod_link">
+      <!-- central box: top length, full height -->
       <visual>
         <origin xyz="0 0 0" rpy="0 0 0"/>
-        <geometry> <box size="${pod_len} ${pod_wid} ${pod_h}"/> </geometry>
+        <geometry> <box size="0.43 ${pod_wid} ${pod_h}"/> </geometry>
         <material name="white"/>
       </visual>
+      <!-- thin bottom plate closing the underside of the full trapezoid footprint -->
+      <visual>
+        <origin xyz="0 0 -0.13" rpy="0 0 0"/>
+        <geometry> <box size="${pod_len} ${pod_wid} 0.02"/> </geometry>
+        <material name="white"/>
+      </visual>
+      <!-- front full-height slant face -->
+      <visual>
+        <origin xyz="0.345 0 0" rpy="0 0.7854 0"/>
+        <geometry> <box size="0.3677 ${pod_wid} 0.005"/> </geometry>
+        <material name="white"/>
+      </visual>
+      <!-- rear full-height slant face -->
+      <visual>
+        <origin xyz="-0.345 0 0" rpy="0 -0.7854 0"/>
+        <geometry> <box size="0.3677 ${pod_wid} 0.005"/> </geometry>
+        <material name="white"/>
+      </visual>
+      <!-- collision: simple full box (slant is visual only) -->
       <collision>
         <origin xyz="0 0 0" rpy="0 0 0"/>
@@ -202,5 +231,5 @@
     <parent link="base_link"/>
     <child  link="top_frame"/>
-    <origin xyz="${pod_len/2 - 0.15} 0 ${pod_z + pod_h/2 + frame_h/2}" rpy="0 0 0"/>
+    <origin xyz="0 0 ${pod_z + pod_h/2 + frame_h/2}" rpy="0 0 0"/>
   </joint>
   <!-- ══════════════════════════════════════════════════════════════
@@ -226,5 +255,5 @@
     <parent link="left_pod_link"/>
     <child  link="mast_link"/>
-    <origin xyz="${pod_len/2 - 0.12} 0 ${pod_h/2 + mast_h/2}" rpy="0 0 0"/>
+    <origin xyz="0.15 0 ${pod_h/2 + mast_h/2}" rpy="0 0 0"/>
   </joint>
   <!-- Comms / control enclosure on the mast (the blue box in the drawing) -->

Commit message: Update sowbot_01.xacro

File: src/agro_robot_sim/urdf/sowbot_01.xacro (robot description, xacro)
@@ -1,6 +1,5 @@
 <?xml version="1.0"?>
 <!--
-  sowbot_urdf.xacro  —
-     • Continuous rubber tracks replace the 4 wheels (visual: long track box + drive/idler rollers)
+    • Continuous rubber tracks replace the 4 wheels (visual: long track box + drive/idler rollers)
     • Chassis split into TWO side body pods sitting above each track
     • Pods joined by a transverse top frame; vertical mast carries GPS / comms / e-stop
@@ -33,6 +32,6 @@
   <xacro:property name="base_link_z"    value="${drive_radius}"/>
   <!-- ── Side body pods (two boxes, one above each track) ── -->
-  <xacro:property name="pod_len"        value="0.95"/>
-  <xacro:property name="pod_wid"        value="0.24"/>
+  <xacro:property name="pod_len"        value="1.10"/>
+  <xacro:property name="pod_wid"        value="0.30"/>
   <xacro:property name="pod_h"          value="0.26"/>
   <!-- pod inner face roughly above the track; centre offset = track_half -->
@@ -158,17 +157,17 @@
        ══════════════════════════════════════════════════════════════ -->
   <xacro:macro name="pod" params="prefix y">
-    <!-- Pod profile: a trapezoid in side view — flat bottom (full 0.95), shorter
-         top (0.43), with a FULL-HEIGHT 45° slant face at each end running from the
+    <!-- Pod profile: a trapezoid in side view — flat bottom (full 1.10), shorter
+         top (0.58), with a FULL-HEIGHT 45° slant face at each end running from the
          bottom-outer edge up to the top-inner edge, so the slant reaches the very
          end of the body. Central box (top length, full height) + two thin slant
-         plates covering the slope faces.
+         plates covering the slope faces. Sized so each track fits within the pod.
          Literals (no math fns / in-macro properties) for parser compatibility:
-           pod_h=0.26, central box len=0.43, slant_len=0.3677, pitch=0.7854 rad,
-           slant centre x=±0.345 (spans bottom-outer 0.475/-0.13 to top-inner 0.215/+0.13) -->
+           pod_h=0.26, central box len=0.58, slant_len=0.3677, pitch=0.7854 rad,
+           slant centre x=±0.42 (spans bottom-outer 0.55/-0.13 to top-inner 0.29/+0.13) -->
     <link name="${prefix}_pod_link">
       <!-- central box: top length, full height -->
       <visual>
         <origin xyz="0 0 0" rpy="0 0 0"/>
-        <geometry> <box size="0.43 ${pod_wid} ${pod_h}"/> </geometry>
+        <geometry> <box size="0.58 ${pod_wid} ${pod_h}"/> </geometry>
         <material name="white"/>
       </visual>
@@ -181,5 +180,5 @@
       <!-- front full-height slant face -->
       <visual>
-        <origin xyz="0.345 0 0" rpy="0 0.7854 0"/>
+        <origin xyz="0.42 0 0" rpy="0 0.7854 0"/>
         <geometry> <box size="0.3677 ${pod_wid} 0.005"/> </geometry>
         <material name="white"/>
@@ -187,5 +186,5 @@
       <!-- rear full-height slant face -->
       <visual>
-        <origin xyz="-0.345 0 0" rpy="0 -0.7854 0"/>
+        <origin xyz="-0.42 0 0" rpy="0 -0.7854 0"/>
         <geometry> <box size="0.3677 ${pod_wid} 0.005"/> </geometry>
         <material name="white"/>

Commit message: Update sowbot_01.xacro reference dimensions and properties

File: src/agro_robot_sim/urdf/sowbot_01.xacro (robot description, xacro)
@@ -1,5 +1,5 @@
 <?xml version="1.0"?>
 <!--
-  Reference dimensions
+  Reference dimensions (from supplied RTU.V4 drawing):
     track ground length   ≈ 1.035 m
     overall body width     ≈ 0.940 m
@@ -31,9 +31,10 @@
   <xacro:property name="pod_len"        value="1.10"/>
   <xacro:property name="pod_wid"        value="0.30"/>
-  <xacro:property name="pod_h"          value="0.26"/>
+  <xacro:property name="pod_h"          value="0.32"/>
   <!-- pod inner face roughly above the track; centre offset = track_half -->
   <xacro:property name="pod_y"          value="${track_half}"/>
-  <!-- pod vertical centre: drop body so its base overlaps the top of the track unit -->
-  <xacro:property name="pod_z"          value="${track_height/2 + pod_h/2 - 0.05}"/>
+  <!-- pod centre: body extends down so its base reaches the track axle centre
+       (base_link z=0), giving the drive/idler axles something to attach to -->
+  <xacro:property name="pod_z"          value="0.16"/>
   <!-- ── Transverse top frame joining the pods ── -->
   <xacro:property name="frame_wid"      value="0.94"/>
@@ -154,35 +155,37 @@
        ══════════════════════════════════════════════════════════════ -->
   <xacro:macro name="pod" params="prefix y">
-    <!-- Pod profile: a trapezoid in side view — flat bottom (full 1.10), shorter
-         top (0.58), with a FULL-HEIGHT 45° slant face at each end running from the
-         bottom-outer edge up to the top-inner edge, so the slant reaches the very
-         end of the body. Central box (top length, full height) + two thin slant
-         plates covering the slope faces. Sized so each track fits within the pod.
+    <!-- Pod profile: VERTICAL lower section (full length 1.10, z -0.16..0) so the
+         body sides clear the track, plus a SLANTED upper section (z 0..+0.16) whose
+         top sets back by the rake at each end — vertical walls below, raked shoulders
+         above, matching the reference. Track top (pod-frame z=-0.05) sits inside the
+         vertical wall, so the track cannot foul the body.
          Literals (no math fns / in-macro properties) for parser compatibility:
-           pod_h=0.26, central box len=0.58, slant_len=0.3677, pitch=0.7854 rad,
-           slant centre x=±0.42 (spans bottom-outer 0.55/-0.13 to top-inner 0.29/+0.13) -->
+           pod_h=0.32; lower box h=0.16 @z=-0.08 (full len 1.10);
+           upper box h=0.16 @z=+0.08 (top len 0.58);
+           upper slant_len=0.3053, pitch=0.5517 rad (~31.6°), centre x=±0.42 z=+0.08
+           (spans shoulder-outer 0.55/0.0 to top-inner 0.29/+0.16) -->
     <link name="${prefix}_pod_link">
-      <!-- central box: top length, full height -->
-      <visual>
-        <origin xyz="0 0 0" rpy="0 0 0"/>
-        <geometry> <box size="0.58 ${pod_wid} ${pod_h}"/> </geometry>
+      <!-- lower vertical box (full length) -->
+      <visual>
+        <origin xyz="0 0 -0.08" rpy="0 0 0"/>
+        <geometry> <box size="${pod_len} ${pod_wid} 0.16"/> </geometry>
         <material name="white"/>
       </visual>
-      <!-- thin bottom plate closing the underside of the full trapezoid footprint -->
-      <visual>
-        <origin xyz="0 0 -0.13" rpy="0 0 0"/>
-        <geometry> <box size="${pod_len} ${pod_wid} 0.02"/> </geometry>
+      <!-- upper central box (top length) -->
+      <visual>
+        <origin xyz="0 0 0.08" rpy="0 0 0"/>
+        <geometry> <box size="0.58 ${pod_wid} 0.16"/> </geometry>
         <material name="white"/>
       </visual>
-      <!-- front full-height slant face -->
-      <visual>
-        <origin xyz="0.42 0 0" rpy="0 0.7854 0"/>
-        <geometry> <box size="0.3677 ${pod_wid} 0.005"/> </geometry>
+      <!-- front upper slant face (shoulder up to top) -->
+      <visual>
+        <origin xyz="0.42 0 0.08" rpy="0 0.5517 0"/>
+        <geometry> <box size="0.3053 ${pod_wid} 0.005"/> </geometry>
         <material name="white"/>
       </visual>
-      <!-- rear full-height slant face -->
-      <visual>
-        <origin xyz="-0.42 0 0" rpy="0 -0.7854 0"/>
-        <geometry> <box size="0.3677 ${pod_wid} 0.005"/> </geometry>
+      <!-- rear upper slant face -->
+      <visual>
+        <origin xyz="-0.42 0 0.08" rpy="0 -0.5517 0"/>
+        <geometry> <box size="0.3053 ${pod_wid} 0.005"/> </geometry>
         <material name="white"/>
       </visual>

Commit message: Update sowbot_01.xacro with new dimensions and features

File: src/agro_robot_sim/urdf/sowbot_01.xacro (robot description, xacro)
@@ -1,5 +1,5 @@
 <?xml version="1.0"?>
 <!--
-  Reference dimensions (from supplied RTU.V4 drawing):
+  Reference dimensions
     track ground length   ≈ 1.035 m
     overall body width     ≈ 0.940 m
@@ -49,4 +49,5 @@
   <material name="black">        <color rgba="0.10 0.10 0.10 1.0"/> </material>
   <material name="grey">         <color rgba="0.55 0.55 0.55 1.0"/> </material>
+  <material name="darkgrey">     <color rgba="0.35 0.35 0.35 1.0"/> </material>
   <material name="orange">       <color rgba="1.00 0.50 0.00 1.0"/> </material>
   <material name="red">          <color rgba="0.80 0.10 0.10 1.0"/> </material>
@@ -154,5 +155,5 @@
        SIDE BODY PODS  (two boxes above the tracks — the split body)
        ══════════════════════════════════════════════════════════════ -->
-  <xacro:macro name="pod" params="prefix y">
+  <xacro:macro name="pod" params="prefix y face">
     <!-- Pod profile: VERTICAL lower section (full length 1.10, z -0.16..0) so the
          body sides clear the track, plus a SLANTED upper section (z 0..+0.16) whose
@@ -190,4 +191,20 @@
         <material name="white"/>
       </visual>
+      <!-- ── Rectangular access hatch (visual only) ───────────────────
+           A single bolt-on access cover on the OUTER side face of the pod
+           (face param: +Y for left pod, -Y for right), light grey, with a
+           small grab handle. Upper-central side, clear of the lower wall and
+           axle mounts (z=-0.16, x=±0.41). Collision stays the full solid box. -->
+      <visual>
+        <origin xyz="0.04 ${face} 0.03" rpy="0 0 0"/>
+        <geometry> <box size="0.30 0.006 0.18"/> </geometry>
+        <material name="grey"/>
+      </visual>
+      <!-- handle: small grab bar standing off the hatch -->
+      <visual>
+        <origin xyz="0.04 ${face*1.18} 0.03" rpy="0 1.5708 0"/>
+        <geometry> <cylinder radius="0.008" length="0.06"/> </geometry>
+        <material name="darkgrey"/>
+      </visual>
       <!-- collision: simple full box (slant is visual only) -->
       <collision>
@@ -206,6 +223,6 @@
     </joint>
   </xacro:macro>
-  <xacro:pod prefix="left"  y=" ${pod_y}"/>
-  <xacro:pod prefix="right" y="-${pod_y}"/>
+  <xacro:pod prefix="left"  y=" ${pod_y}" face=" 0.152"/>
+  <xacro:pod prefix="right" y="-${pod_y}" face="-0.152"/>
   <!-- ══════════════════════════════════════════════════════════════
        TOP FRAME  (transverse bar joining the two pods)
@@ -273,5 +290,5 @@
     <origin xyz="0.07 0 0.05" rpy="0 0 0"/>
   </joint>
-  <!-- E-stop button (the red mushroom on the side) -->
+  <!-- E-stop button (red mushroom) on the front face -->
   <link name="estop_link">
     <visual>
@@ -284,5 +301,5 @@
     <parent link="left_pod_link"/>
     <child  link="estop_link"/>
-    <origin xyz="${pod_len/2 - 0.20} ${pod_wid/2} 0.02" rpy="0 0 0"/>
+    <origin xyz="${pod_len/2 + 0.015} 0 -0.05" rpy="0 0 0"/>
   </joint>
   <!-- ══════════════════════════════════════════════════════════════
